File: _saved_Spot_Welder_Hardware.sch (KiCad schematic (older format))
At the start: 148 parts, among them J1 Mini USB, J2 Conn_01x03_Male, Q1 Q_NMOS_GSD, Q10 Q_NMOS_GDS, Q11 Q_NMOS_GDS, Q12 Q_NMOS_GDS, Q13 Q_NMOS_GDS, Q2 MBT3904, Q3 Q_NMOS_GDS, Q4 Q_NMOS_GDS, Q5 Q_NMOS_GDS, Q6 Q_NMOS_GDS, Q7 Q_NMOS_GDS, Q8 Q_NMOS_GDS, Q9 Q_NMOS_GDS, SW1 SW_Push, SW2 SW_SPDT, SW3 Lead Voltage Trigger, SW4 SW_Push, U1 OKI, U2 ATMEGA328P, U3 FAN3122TMXCT-ND, U4 FT232RL, U5 FAN3122TMXCT-ND, Y1 Crystal

Commit message: Finished Silkscreen
Changed lines of the file:
@@
 Text Notes 6750 5900 0    20   ~ 0
 Used to toggle\nlead voltage trigger mode
+Text GLabel 10400 5200 2    60   Input ~ 0
+5V_Ind
+Text GLabel 10400 5300 2    60   Input ~ 0
+7.5V_Ind
+Text GLabel 10400 5400 2    60   Input ~ 0
+10V_Ind
 Text GLabel 10400 5500 2    60   Input ~ 0
-5V_Ind
-Text GLabel 10400 5400 2    60   Input ~ 0
-7.5V_Ind
-Text GLabel 10400 5300 2    60   Input ~ 0
-10V_Ind
-Text GLabel 10400 5200 2    60   Input ~ 0
 12.5V_Ind
+Text Notes 10900 5550 0    60   ~ 0
+D12
 Text Notes 10900 5450 0    60   ~ 0
-D12
+D11
 Text Notes 10900 5350 0    60   ~ 0
-D11
+D10
 Text Notes 10900 5250 0    60   ~ 0
-D10
-Text Notes 10900 5150 0    60   ~ 0
 D9
 Text GLabel 10400 7300 2    60   Input ~ 0
