File: Spot_Welder_Hardware.kicad_pcb (KiCad board)
At the start: 2 copper layers, 268.7 x 183.1 mm, 155 parts, among them J1 Mini USB, J2 Conn_01x03_Male, Q1 Q_NMOS_GSD, Q10 Q_NMOS_GDS, Q11 Q_NMOS_GDS, Q12 Q_NMOS_GDS, Q13 Q_NMOS_GDS, Q2 MBT3904, Q3 Q_NMOS_GDS, Q4 Q_NMOS_GDS, Q5 Q_NMOS_GDS, Q6 Q_NMOS_GDS, Q7 Q_NMOS_GDS, Q8 Q_NMOS_GDS, Q9 Q_NMOS_GDS, SW1 SW_Push, SW2 SW_SPDT, SW3 Lead Voltage Trigger, SW4 SW_Push, U1 OKI, U2 ATMEGA328P, U3 FAN3122TMXCT-ND, U4 FT232RL, U5 FAN3122TMXCT-ND, Y1 Crystal

Commit message: Moved around ground planes
Routing:
- net +5V: track 127.1 -> 156.4 mm, vias 4 -> 8
- net VS: track 104.9 -> 101.8 mm
- net GND: track 176.4 -> 174.8 mm
- net Pulse_Out: track 270.2 -> 271.3 mm, vias 5 -> 2

Commit message: Routed Ground Plane
Routing:
- net GND: track 174.8 -> 156.4 mm, vias 42 -> 43
- net Pulse_Out: track 271.3 -> 271.5 mm, vias 2 -> 4
Changed lines of the file:
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@@
     (thickness 1.6)
     (drawings 40)
-    (tracks 572)
+    (tracks 577)
     (zones 0)
     (modules 155)
@@
   (segment (start 42.072 191.936) (end 39.712 191.936) (width 0.381) (layer F.Cu) (net 4))
   (segment (start 39.712 191.936) (end 39.624 192.024) (width 0.381) (layer F.Cu) (net 4))
-  (segment (start 78.318 128.102) (end 74.422 124.206) (width 1.27) (layer F.Cu) (net 4))
-  (segment (start 78.318 142.494) (end 78.318 128.102) (width 1.27) (layer F.Cu) (net 4))
   (via (at 109.982 169.672) (size 0.6) (drill 0.4) (layers F.Cu B.Cu) (net 4))
   (segment (start 109.982 168.016) (end 109.982 169.672) (width 0.381) (layer F.Cu) (net 4))
@@
   (segment (start 62.461 178.285) (end 62.738 178.562) (width 0.381) (layer F.Cu) (net 4))
   (segment (start 141.732 187.071) (end 147.066 187.071) (width 1.27) (layer B.Cu) (net 4))
+  (via (at 78.486 140.97) (size 0.6) (drill 0.4) (layers F.Cu B.Cu) (net 4))
+  (segment (start 78.318 142.494) (end 78.318 141.138) (width 0.381) (layer F.Cu) (net 4))
+  (segment (start 78.318 141.138) (end 78.486 140.97) (width 0.381) (layer F.Cu) (net 4))
   (segment (start 121.412 167.386) (end 125.222 167.386) (width 0.381) (layer F.Cu) (net 5))
   (segment (start 109.982 166.116) (end 113.792 169.926) (width 0.381) (layer F.Cu) (net 6))
@@
   (segment (start 242.480501 189.902501) (end 242.189 189.611) (width 0.381) (layer F.Cu) (net 60))
   (segment (start 242.57 189.992) (end 242.189 189.611) (width 0.381) (layer F.Cu) (net 60))
-  (segment (start 242.57 194.183) (end 242.57 189.992) (width 0.381) (layer F.Cu) (net 60))
-  (segment (start 241.681 195.072) (end 242.57 194.183) (width 0.381) (layer F.Cu) (net 60))
   (segment (start 146.939 195.072) (end 241.681 195.072) (width 0.381) (layer F.Cu) (net 60))
   (segment (start 146.304 187.071) (end 146.304 194.437) (width 0.381) (layer F.Cu) (net 60))
   (segment (start 146.304 194.437) (end 146.939 195.072) (width 0.381) (layer F.Cu) (net 60))
+  (via (at 242.57 194.31) (size 0.6) (drill 0.4) (layers F.Cu B.Cu) (net 60))
+  (segment (start 241.681 195.072) (end 241.808 195.072) (width 0.381) (layer F.Cu) (net 60))
+  (segment (start 241.808 195.072) (end 242.57 194.31) (width 0.381) (layer F.Cu) (net 60))
+  (via (at 242.480501 189.902501) (size 0.6) (drill 0.4) (layers F.Cu B.Cu) (net 60))
+  (segment (start 242.57 194.31) (end 242.57 189.992) (width 0.381) (layer B.Cu) (net 60))
+  (segment (start 242.57 189.992) (end 242.480501 189.902501) (width 0.381) (layer B.Cu) (net 60))
   (segment (start 121.412 180.086) (end 126.746 180.086) (width 0.381) (layer F.Cu) (net 61))
   (segment (start 127.762 181.102) (end 127.762 187.706) (width 0.381) (layer F.Cu) (net 61))
@@
     (polygon
       (pts
-        (xy 54.356 139.446) (xy 145.796 139.446) (xy 145.796 196.596) (xy 282.956 196.596) (xy 282.956 13.716)
-        (xy 14.224 13.716) (xy 14.224 132.334) (xy 54.356 132.334)
+        (xy 54.356 139.446) (xy 71.374 139.446) (xy 71.374 121.158) (xy 77.47 121.158) (xy 77.47 139.446)
+        (xy 145.796 139.446) (xy 145.796 196.596) (xy 282.956 196.596) (xy 282.956 13.716) (xy 14.224 13.716)
+        (xy 14.224 132.334) (xy 54.356 132.334)
       )
     )
@@
     (polygon
       (pts
-        (xy 14.224 182.88) (xy 54.356 182.88) (xy 54.356 139.954) (xy 145.288 139.954) (xy 145.288 196.596)
-        (xy 14.224 196.596)
+        (xy 14.224 182.88) (xy 54.356 182.88) (xy 54.356 139.954) (xy 71.882 139.954) (xy 71.882 121.666)
+        (xy 76.962 121.666) (xy 76.962 139.954) (xy 145.288 139.954) (xy 145.288 196.596) (xy 14.224 196.596)
       )
     )

Commit message: Updated 6-32 Hole Size
Parts:
- removed the REF** at (19.3, 18.8)
- removed the REF** at (277.9, 18.5)
- added REF**: 6-32 Screw Hole, Project Library:6-32 Screw Hole, F.Cu at (20.6, 17.5)
- added REF**: 6-32 Screw Hole, Project Library:6-32 Screw Hole, F.Cu at (276.6, 17.3)
- moved REF** 1.80 mm to (274.6, 192.8)
- moved REF** 1.80 mm to (11.4, 199.4)
Other:
- board size 268.7 x 183.1 mm -> 263.7 x 182.9 mm
Changed lines of the file:
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@@
   )
   (setup
-    (last_trace_width 0.381)
+    (last_trace_width 2.54)
     (user_trace_width 0.254)
     (user_trace_width 0.381)
@@
   )
   (module "Project Library:6-32 Screw Hole" (layer F.Cu)
-    (at 10.16 198.12 90)
+    (at 11.43 199.39 90)
     (fp_text reference REF** (at 0 0.5 90) (layer F.SilkS) hide
       (effects (font (size 1 1) (thickness 0.15)))
@@
   )
   (module "Project Library:6-32 Screw Hole" (layer F.Cu)
-    (at 19.304 18.796)
+    (at 20.574 17.526)
     (fp_text reference REF** (at 0 0.5) (layer F.SilkS) hide
       (effects (font (size 1 1) (thickness 0.15)))
@@
   )
   (module "Project Library:6-32 Screw Hole" (layer F.Cu)
-    (at 275.844 191.516 180)
+    (at 274.574 192.786 180)
     (fp_text reference REF** (at 0 0.5 180) (layer F.SilkS) hide
       (effects (font (size 1 1) (thickness 0.15)))
@@
   )
   (module "Project Library:6-32 Screw Hole" (layer F.Cu)
-    (at 277.876 18.542 270)
+    (at 276.606 17.272 270)
     (fp_text reference REF** (at 0 0.5 270) (layer F.SilkS) hide
       (effects (font (size 1 1) (thickness 0.15)))
@@
     )
   )
-  (gr_line (start 14.224 18.796) (end 14.224 191.516) (layer Edge.Cuts) (width 0.15))
-  (gr_line (start 19.304 196.596) (end 277.876 196.596) (layer Edge.Cuts) (width 0.15))
-  (gr_arc (start 19.304 191.516) (end 14.224 191.516) (angle -90) (layer Edge.Cuts) (width 0.15))
-  (gr_circle (center 19.304 191.516) (end 14.224 191.516) (layer F.SilkS) (width 0.2))
-  (gr_line (start 277.876 13.462) (end 19.304 13.716) (layer Edge.Cuts) (width 0.15))
-  (gr_circle (center 19.304 18.796) (end 19.304 13.716) (layer F.SilkS) (width 0.2))
-  (gr_arc (start 19.304 18.796) (end 19.304 13.716) (angle -90) (layer Edge.Cuts) (width 0.15))
-  (gr_line (start 282.956 191.516) (end 282.956 18.542) (layer Edge.Cuts) (width 0.15))
-  (gr_circle (center 277.876 191.516) (end 277.876 196.596) (layer F.SilkS) (width 0.2))
-  (gr_arc (start 277.876 191.516) (end 277.876 196.596) (angle -90) (layer Edge.Cuts) (width 0.15))
-  (gr_circle (center 277.876 18.542) (end 282.956 18.542) (layer F.SilkS) (width 0.2))
-  (gr_arc (start 277.876 18.542) (end 282.956 18.542) (angle -90) (layer Edge.Cuts) (width 0.15))
+  (gr_arc (start 276.606 192.786) (end 276.606 196.596) (angle -90) (layer Edge.Cuts) (width 0.15))
+  (gr_line (start 20.574 196.596) (end 276.606 196.596) (layer Edge.Cuts) (width 0.15))
+  (gr_arc (start 20.574 192.786) (end 16.764 192.786) (angle -90) (layer Edge.Cuts) (width 0.15))
+  (gr_line (start 16.764 17.526) (end 16.764 192.786) (layer Edge.Cuts) (width 0.15))
+  (gr_arc (start 20.574 17.526) (end 20.574 13.716) (angle -90) (layer Edge.Cuts) (width 0.15))
+  (gr_line (start 20.574 13.716) (end 276.606 13.716) (layer Edge.Cuts) (width 0.15))
+  (gr_line (start 280.416 17.526) (end 280.416 192.786) (layer Edge.Cuts) (width 0.15))
+  (gr_arc (start 276.606 17.526) (end 280.416 17.526) (angle -90) (layer Edge.Cuts) (width 0.15))
+  (gr_circle (center 20.574 192.786) (end 24.384 192.786) (layer F.SilkS) (width 0.2))
+  (gr_circle (center 20.574 17.526) (end 24.384 17.526) (layer F.SilkS) (width 0.2))
+  (gr_circle (center 276.606 192.786) (end 280.416 192.786) (layer F.SilkS) (width 0.2))
+  (gr_circle (center 276.606 17.526) (end 280.416 17.526) (layer F.SilkS) (width 0.2))
   (gr_text DTR (at 71.628 188.976) (layer F.SilkS)
     (effects (font (size 1.5 1.5) (thickness 0.3)))

Commit message: Mino changes from Assembly
Parts:
- moved D11 5.69 mm to (50.3, 155.5), turned to 270 degrees
Connections:
- REF** pad 1: GND -> V+
Routing:
- net Net-(D11-Pad1): track 17.8 -> 11.0 mm
- net V+: track 24.6 -> 24.1 mm
Other:
- board text added: "L PWR"
- board text added: "Over Voltage"
- board text added: "Plse"
- board text added: "X Trg"
Changed lines of the file:
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@@
   (general
     (thickness 1.6)
-    (drawings 40)
-    (tracks 577)
+    (drawings 42)
+    (tracks 575)
     (zones 0)
     (modules 155)
@@
   )
   (setup
-    (last_trace_width 2.54)
+    (last_trace_width 0.381)
     (user_trace_width 0.254)
     (user_trace_width 0.381)
@@
     (mod_text_size 1 1)
     (mod_text_width 0.15)
-    (pad_size 3.683 3.683)
-    (pad_drill 0.762)
+    (pad_size 2.3 1.7)
+    (pad_drill 1.5)
     (pad_to_mask_clearance 0.2)
     (aux_axis_origin 0 0)
     (visible_elements 7FFFFFFF)
     (pcbplotparams
-      (layerselection 0x00030_80000001)
+      (layerselection 0x010fc_ffffffff)
       (usegerberextensions false)
       (usegerberattributes false)
@@
       (outputformat 1)
       (mirror false)
-      (drillshape 1)
+      (drillshape 0)
       (scaleselection 1)
-      (outputdirectory ""))
+      (outputdirectory "Gerbs/"))
   )
   (net 0 "")
@@
     )
     (pad 1 thru_hole circle (at 0 0.0254) (size 18.288 18.288) (drill 9.144) (layers *.Cu *.Mask)
-      (net 4 GND))
+      (net 3 V+))
   )
   (module MRDT_Devices:BUZZER_SMI_1324_TW_5V_2_R (layer F.Cu)
@@
   )
   (module LEDs:LED_0603_HandSoldering (layer F.Cu)
-    (at 48.852 161.036 180)
+    (at 50.292 155.532 270)
     (descr "LED SMD 0603, hand soldering")
     (tags "LED 0603")
     (attr smd)
-    (fp_text reference D11 (at 0 -1.45 180) (layer F.SilkS)
+    (fp_text reference D11 (at 0 -1.45 270) (layer F.SilkS)
       (effects (font (size 1 1) (thickness 0.15)))
     )
-    (fp_text value "Over Voltage" (at 0 1.55 180) (layer F.Fab)
+    (fp_text value "Over Voltage" (at 0 1.55 270) (layer F.Fab)
       (effects (font (size 1 1) (thickness 0.15)))
     )
@@
     (fp_line (start 1.95 0.7) (end -1.96 0.7) (layer F.CrtYd) (width 0.05))
     (fp_line (start -0.8 -0.4) (end -0.8 0.4) (layer F.Fab) (width 0.1))
-    (pad 1 smd rect (at -1.1 0 180) (size 1.2 0.9) (layers F.Cu F.Paste F.Mask)
+    (pad 1 smd rect (at -1.1 0 270) (size 1.2 0.9) (layers F.Cu F.Paste F.Mask)
       (net 73 "Net-(D11-Pad1)"))
-    (pad 2 smd rect (at 1.1 0 180) (size 1.2 0.9) (layers F.Cu F.Paste F.Mask)
+    (pad 2 smd rect (at 1.1 0 270) (size 1.2 0.9) (layers F.Cu F.Paste F.Mask)
       (net 3 V+))
     (model ${KISYS3DMOD}/LEDs.3dshapes/LED_0603.wrl
@@
       (effects (font (size 1 1) (thickness 0.15)))
     )
-    (fp_line (start -3.3 6.35) (end 3.3 6.35) (layer F.SilkS) (width 0.15))
-    (fp_line (start 3.3 -6.35) (end -3.3 -6.35) (layer F.SilkS) (width 0.15))
-    (fp_line (start -3.3 6.35) (end -3.3 -6.35) (layer F.SilkS) (width 0.15))
     (fp_line (start 3.3 6.35) (end 3.3 -6.35) (layer F.SilkS) (width 0.15))
-    (pad 1 thru_hole oval (at 0 -4.7) (size 2.2 1.6) (drill oval 1.4 0.9) (layers *.Cu *.Mask)
-      (net 65 "Net-(R12-Pad2)"))
-    (pad 2 thru_hole oval (at 0 0) (size 2.2 1.6) (drill oval 1.4 0.9) (layers *.Cu *.Mask)
-      (net 24 Power_GND))
-    (pad 3 thru_hole oval (at 0 4.7) (size 2.2 1.6) (drill oval 1.4 0.9) (layers *.Cu *.Mask)
+    (fp_line (start -3.3 6.35) (end -3.3 -6.35) (layer F.SilkS) (width 0.15))
+    (fp_line (start 3.3 -6.35) (end -3.3 -6.35) (layer F.SilkS) (width 0.15))
+    (fp_line (start -3.3 6.35) (end 3.3 6.35) (layer F.SilkS) (width 0.15))
+    (pad 3 thru_hole oval (at 0 4.7) (size 2.3 1.7) (drill oval 1.5 1) (layers *.Cu *.Mask)
       (net 12 Conn_GND))
+    (pad 2 thru_hole oval (at 0 0) (size 2.3 1.7) (drill oval 1.5 1) (layers *.Cu *.Mask)
+      (net 24 Power_GND))
+    (pad 1 thru_hole oval (at 0 -4.7) (size 2.3 1.7) (drill oval 1.5 1) (layers *.Cu *.Mask)
+      (net 65 "Net-(R12-Pad2)"))
   )
   (module "Project Library:SPST_DIP_Switch" (layer F.Cu)
@@
     )
   )
+  (gr_text "Over\nVoltage" (at 52.832 160.02) (layer F.SilkS)
+    (effects (font (size 1.5 1.5) (thickness 0.3)))
+  )
+  (gr_text GND (at 44.196 160.528) (layer F.SilkS)
+    (effects (font (size 2.54 2.54) (thickness 0.508)))
+  )
+  (gr_text V+ (at 44.196 152.654) (layer F.SilkS)
+    (effects (font (size 2.54 2.54) (thickness 0.508)))
+  )
   (gr_arc (start 276.606 192.786) (end 276.606 196.596) (angle -90) (layer Edge.Cuts) (width 0.15))
   (gr_line (start 20.574 196.596) (end 276.606 196.596) (layer Edge.Cuts) (width 0.15))
@@
     (effects (font (size 1.5 1.5) (thickness 0.3)) (justify left))
   )
-  (gr_text GND (at 257.048 192.532) (layer F.SilkS)
+  (gr_text V+ (at 257.048 192.532) (layer F.SilkS)
     (effects (font (size 5.08 5.08) (thickness 1.016)))
   )
@@
     (effects (font (size 1.5 1.5) (thickness 0.3)) (justify left))
   )
-  (gr_text PWR (at 105.156 186.944 90) (layer F.SilkS)
+  (gr_text "X Trg" (at 105.156 186.944 90) (layer F.SilkS)
     (effects (font (size 1.5 1.5) (thickness 0.3)) (justify left))
   )
-  (gr_text TX (at 99.822 186.69 90) (layer F.SilkS)
+  (gr_text "L PWR" (at 99.822 186.69 90) (layer F.SilkS)
     (effects (font (size 1.5 1.5) (thickness 0.3)) (justify left))
   )
-  (gr_text RX (at 102.362 186.944 90) (layer F.SilkS)
+  (gr_text Plse (at 102.362 186.944 90) (layer F.SilkS)
     (effects (font (size 1.5 1.5) (thickness 0.3)) (justify left))
   )
@@
     (effects (font (size 2.54 2.54) (thickness 0.508)) (justify left))
   )
-  (gr_line (start -91.44 254) (end -91.44 -254) (layer F.SilkS) (width 0.2))
   (segment (start 68.326 148.336) (end 67.691 147.701) (width 0.381) (layer F.Cu) (net 1))
   (segment (start 70.866 148.336) (end 68.326 148.336) (width 0.381) (layer F.Cu) (net 1))
@@
   (segment (start 145.542 158.056) (end 145.542 163.766) (width 0.381) (layer F.Cu) (net 2))
   (segment (start 86.866 142.494) (end 86.866 138.178) (width 1.27) (layer F.Cu) (net 3))
-  (segment (start 47.371 160.655) (end 47.752 161.036) (width 0.381) (layer F.Cu) (net 3))
   (segment (start 133.419 156.886) (end 135.042 155.263) (width 0.381) (layer F.Cu) (net 3))
   (segment (start 132.588 156.886) (end 133.419 156.886) (width 0.381) (layer F.Cu) (net 3))
@@
   (segment (start 67.691 142.621) (end 70.231 142.621) (width 0.381) (layer F.Cu) (net 72))
   (segment (start 83.566 142.494) (end 80.518 142.494) (width 1.27) (layer F.Cu) (net 72))
-  (segment (start 50.292 160.696) (end 49.952 161.036) (width 0.381) (layer F.Cu) (net 73))
-  (segment (start 50.292 147.742) (end 50.292 160.696) (width 0.381) (layer F.Cu) (net 73))
-  (segment (start 50.292 147.742) (end 50.292 143.424) (width 0.381) (layer F.Cu) (net 73))
+  (segment (start 50.292 144.405) (end 50.292 154.432) (width 0.381) (layer F.Cu) (net 73))
+  (segment (start 50.292 143.424) (end 50.292 144.405) (width 0.381) (layer F.Cu) (net 73))
   (zone (net 25) (net_name VS) (layer F.Cu) (hatch edge 0.508)
     (connect_pads yes (clearance 0.508))

Commit message: Fixed Layout
Parts:
- added G***: LOGO, MRDT_Silkscreens:Andrew_Van_Horn_Sig_15mm, F.Cu at (240.2, 157.3)
- added R41: 1000, Resistors_SMD:R_0603_HandSoldering, F.Cu at (109.0, 180.2)
- added R42: 1000, Resistors_SMD:R_0603_HandSoldering, F.Cu at (110.9, 189.0)
Routing:
- net GND: track 156.4 -> 168.5 mm, vias 43 -> 44
- net +5V: track 156.4 -> 163.4 mm, vias 8 -> 10
- net Lead_Voltage_Trigger: track 10.3 -> 13.7 mm
- net Pulse_Out: track 271.5 -> 273.6 mm
Other:
- board text added: "Spot Welder, Rev 2 Mars Rover Design Team, 2019 Missouri S&T Andrew Van Horn With help from Robert Ruark"
- board text removed: "Spot Welder, Rev 1 Mars Rover Design Team, 2019 Missouri S&T Andrew Van Horn In Conjunction with Robert Ruark"

Commit message: Fixed Layout Issues
Parts:
- turned SW2 to 180 degrees
Routing:
- net Net-(R12-Pad2): track 8.43 -> 19.0 mm
- net Conn_GND: track 56.0 -> 65.3 mm
Other:
- board text added: "Over Voltage (15V)"
- board text removed: "L PWR"
- board text removed: "Over Voltage"

Commit message: Added ToDo Notes
Routing:
- net GND: track 168.5 -> 165.3 mm
Changed lines of the file:
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@@
     (thickness 1.6)
     (drawings 42)
-    (tracks 600)
+    (tracks 599)
     (zones 0)
     (modules 158)
@@
   (segment (start 150.289 189.611) (end 150.289 189.611) (width 0.762) (layer F.Cu) (net 4))
   (via (at 150.289 189.611) (size 0.6) (drill 0.4) (layers F.Cu B.Cu) (net 4))
-  (segment (start 70.866 145.288) (end 74.041 145.288) (width 0.381) (layer F.Cu) (net 4))
   (segment (start 246.126 191.77) (end 246.126 191.77) (width 0.762) (layer F.Cu) (net 4))
   (segment (start 243.84 191.77) (end 246.126 191.77) (width 0.762) (layer F.Cu) (net 4))
