File: SpotWelder_Hardware/Spot_Welder_Hardware.sch (KiCad schematic (older format))
At the start: 150 parts, among them J1 Mini USB, J2 Conn_01x03_Male, Q1 Q_NMOS_GSD, Q10 Q_NMOS_GDS, Q11 Q_NMOS_GDS, Q12 Q_NMOS_GDS, Q13 Q_NMOS_GDS, Q2 MBT3904, Q3 Q_NMOS_GDS, Q4 Q_NMOS_GDS, Q5 Q_NMOS_GDS, Q6 Q_NMOS_GDS, Q7 Q_NMOS_GDS, Q8 Q_NMOS_GDS, Q9 Q_NMOS_GDS, SW1 SW_Push, SW2 SW_SPDT, SW3 Lead Voltage Trigger, SW4 SW_Push, U1 OKI, U2 ATMEGA328P, U3 FAN3122TMXCT-ND, U4 FT232RL, U5 FAN3122TMXCT-ND, Y1 Crystal

Commit message: Changed OverV sense zener to 14V to provide better tolerance after testing.
Parts:
- D10: value 15V -> 14V
- J1: symbol conn:Conn_01x05 -> Connector:Conn_01x05_Male
- J2: symbol conn:Conn_01x03_Male -> Connector:Conn_01x03_Male
- Q2: symbol transistors:2N2219 -> Transistor_BJT:MMBT3904
- SW1: symbol switches:SW_Push -> Switch:SW_Push
- SW2: symbol switches:SW_SPDT -> Switch:SW_SPDT
- SW3: symbol switches:SW_SPST -> Switch:SW_SPST
Connections:
- no-connect marks 0 -> 1
Changed lines of the file:
@@
 Interface
 $Comp
-L switches:SW_SPST SW3
+L Switch:SW_SPST SW3
 U 1 1 5B37438C
 P 5800 5750
@@
 $EndComp
 $Comp
-L conn:Conn_01x05 J1
+L Connector:Conn_01x05_Male J1
 U 1 1 5B3A46C1
 P 6500 3850
@@
 F 4 "151-1206-1-ND" H 6500 3850 60  0001 C CNN "Part Number"
 	1    6500 3850
-	-1   0    0    -1
+	1    0    0    -1
 $EndComp
 Text GLabel 6700 3650 2    60   Output ~ 0
@@
 D7
 $Comp
-L switches:SW_Push SW1
+L Switch:SW_Push SW1
 U 1 1 5B36DB85
 P 4600 5750
@@
 	9700 1900 9700 4550
 $Comp
-L switches:SW_SPDT SW2
+L Switch:SW_SPDT SW2
 U 1 1 5B3B77AE
 P 5050 5200
@@
 Power_GND
 $Comp
-L transistors:2N2219 Q2
+L Transistor_BJT:MMBT3904 Q2
 U 1 1 5B3E4E66
 P 8800 2950
@@
 P 8050 2800
 F 0 "D10" H 8050 2900 50  0000 C CNN
-F 1 "15V" H 8050 2700 50  0000 C CNN
+F 1 "14V" H 8050 2700 50  0000 C CNN
 F 2 "Diodes_SMD:D_SOD-123" H 8050 2800 50  0001 C CNN
 F 3 "" H 8050 2800 50  0001 C CNN
@@
 DTR
 $Comp
-L conn:Conn_01x03_Male J2
+L Connector:Conn_01x03_Male J2
 U 1 1 5B598051
 P 6450 3050
@@
 Wire Wire Line
 	4800 5750 4850 5750
-Connection ~ 4800 5750
 Wire Notes Line
 	4100 6050 7200 6050
@@
 	0    1    1    0
 $EndComp
+NoConn ~ 6700 3950
 $EndSCHEMATC
